Commit message: Imported the robot into Gazebo but could not get controls to work for the robot, needs more debugging.

File: justbaked/install/robdesc/share/robdesc/description/robot.urdf.xacro (robot description, xacro)
@@ -1 +1,5 @@
-/home/jack/justbaked/justbaked/src/robdesc/description/robot.urdf.xacro
+<?xml version="1.0"?>
+<robot xmlns:xacro="http://www.ros.org/wiki/xacro" name="justbaked">
+    <xacro:include filename="robotcore.xacro"/>
+    <xacro:include filename="mobile.gazebo"/>
+</robot>

File: justbaked/install/robdesc/share/robdesc/description/robotcore.xacro (robot description, xacro)
@@ -1 +1,148 @@
-/home/jack/justbaked/justbaked/src/robdesc/description/robotcore.xacro
+<?xml version="1.0"?>
+<robot xmlns:xacro="http://www.ros.org/wiki/xacro">
+<link name="base_link">
+</link>
+<!-- Chassis  -->
+<joint name="chassis_joint" type="fixed">
+    <origin xyz="-0.1 0.0 0.05"/>
+    <parent link="base_link"/>
+    <child link="chassis"/>
+</joint>
+<link name="chassis">
+    <visual name="chassis">
+        <origin xyz="0.0 0.0 0.16666665" rpy="0.0 0.0 0.0"/>
+        <geometry>
+            <box size="1.0 0.8 0.3333333"/>
+        </geometry>
+        <material name="red">
+            <color rgba="1.0 0.0 0.0 1.0"/>
+        </material>
+    </visual>
+    <collision>
+        <origin xyz="0.0 0.0 0.05" rpy="0.0 0.0 0.0"/>
+        <geometry>
+            <box size="1.0 1.0 0.3333333"/>
+        </geometry>
+    </collision>
+    <inertial>
+        <origin xyz="0.0 0.0 0.16666665" rpy="0.0 0.0 0.0"/>
+        <mass value="10.0"/>
+        <inertia ixx="0.625924" ixy="0" ixz="0" iyy="1.36667" iyz="0" izz="0.92592"/>
+    </inertial>
+</link>
+<!-- Front left wheel -->
+<joint name="front_left_wheel_joint" type="continuous">
+    <origin xyz="0.4 0.45 0.05" rpy="${pi/2} 0.0 0.0"/>
+    <parent link="chassis"/>
+    <child link="front_left_wheel"/>
+    <axis xyz="0.0 0.0 1.0"/>
+</joint>
+<link name="front_left_wheel">
+    <visual name="front_left_wheel">
+        <origin xyz="0.0 0.0 0.0" rpy="0.0 0.0 0.0"/>
+        <geometry>
+            <cylinder radius="0.1" length="0.1"/>
+        </geometry>
+        <material name="black">
+            <color rgba="0.0 0.0 0.0 1.0"/>
+        </material>
+    </visual>
+    <inertial>
+        <origin xyz="0.0 0.0 0.0" rpy="0.0 0.0 0.0"/>
+        <mass value="1.0"/>
+        <inertia ixx="0.003333333" ixy="0" ixz="0" iyy="0.003333333" iyz="0" izz="0.005"/>
+    </inertial>
+</link>
+<!-- Rear left wheel -->
+<joint name="rear_left_wheel_joint" type="continuous">
+    <origin xyz="-0.4 0.45 0.05" rpy="${pi/2} 0.0 0.0"/>
+    <parent link="chassis"/>
+    <child link="rear_left_wheel"/>
+    <axis xyz="0.0 0.0 1.0"/>
+</joint>
+<link name="rear_left_wheel">
+    <visual name="rear_left_wheel">
+        <origin xyz="0.0 0.0 0.0" rpy="0.0 0.0 0.0"/>
+        <geometry>
+            <cylinder radius="0.1" length="0.1"/>
+        </geometry>
+        <material name="black">
+            <color rgba="0.0 0.0 0.0 1.0"/>
+        </material>
+    </visual>
+    <inertial>
+        <origin xyz="0.0 0.0 0.0" rpy="0.0 0.0 0.0"/>
+        <mass value="1.0"/>
+        <inertia ixx="0.003333333" ixy="0" ixz="0" iyy="0.003333333" iyz="0" izz="0.005"/>
+    </inertial>
+</link>
+<!-- Front right wheel -->
+<joint name="front_right_wheel_joint" type="continuous">
+    <origin xyz="0.4 -0.45 0.05" rpy="${pi/2} 0.0 0.0"/>
+    <parent link="chassis"/>
+    <child link="front_right_wheel"/>
+    <axis xyz="0.0 0.0 1.0"/>
+</joint>
+<link name="front_right_wheel">
+    <visual name="front_right_wheel">
+        <origin xyz="0.0 0.0 0.0" rpy="0.0 0.0 0.0"/>
+        <geometry>
+            <cylinder radius="0.1" length="0.1"/>
+        </geometry>
+        <material name="black">
+            <color rgba="0.0 0.0 0.0 1.0"/>
+        </material>
+    </visual>
+    <inertial>
+        <origin xyz="0.0 0.0 0.0" rpy="0.0 0.0 0.0"/>
+        <mass value="1.0"/>
+        <inertia ixx="0.003333333" ixy="0" ixz="0" iyy="0.003333333" iyz="0" izz="0.005"/>
+    </inertial>
+</link>
+<!-- Rear right wheel -->
+<joint name="rear_right_wheel_joint" type="continuous">
+    <origin xyz="-0.4 -0.45 0.05" rpy="${pi/2} 0.0 0.0"/>
+    <parent link="chassis"/>
+    <child link="rear_right_wheel"/>
+    <axis xyz="0.0 0.0 1.0"/>
+</joint>
+<link name="rear_right_wheel">
+    <visual name="rear_right_wheel">
+        <origin xyz="0.0 0.0 0.0" rpy="0.0 0.0 0.0"/>
+        <geometry>
+            <cylinder radius="0.1" length="0.1"/>
+        </geometry>
+        <material name="black">
+            <color rgba="0.0 0.0 0.0 1.0"/>
+        </material>
+    </visual>
+    <inertial>
+        <origin xyz="0.0 0.0 0.0" rpy="0.0 0.0 0.0"/>
+        <mass value="1.0"/>
+        <inertia ixx="0.003333333" ixy="0" ixz="0" iyy="0.003333333" iyz="0" izz="0.005"/>
+    </inertial>
+</link>
+<!-- Lidar -->
+<joint name="lidar_joint" type="continuous">
+    <origin xyz="0.0 0.0 0.3661417" rpy="0.0 0.0 0.0"/>
+    <parent link="chassis"/>
+    <child link="lidar"/>
+    <axis xyz="0.0 0.0 1.0"/>
+</joint>
+<link name="lidar">
+    <visual name="lidar">
+        <origin xyz="0.0 0.0 0.0" rpy="0.0 0.0 0.0"/>
+        <geometry>
+            <cylinder radius="0.229659" length="0.0656168"/>
+        </geometry>
+        <material name="white">
+            <color rgba="1.0 1.0 1.0 1.0"/>
+        </material>
+    </visual>
+    <inertial>
+        <origin xyz="0.0 0.0 0.0" rpy="0.0 0.0 0.0"/>
+        <mass value="1.0"/>
+        <inertia ixx="0.013544611" ixy="0" ixz="0" iyy="0.013544611" iyz="0" izz="0.026371628"/>
+    </inertial>
+</link>
+</robot>

File: justbaked/src/robdesc/description/robot.urdf.xacro (robot description, xacro)
@@ -2,3 +2,4 @@
 <robot xmlns:xacro="http://www.ros.org/wiki/xacro" name="justbaked">
     <xacro:include filename="robotcore.xacro"/>
+    <xacro:include filename="mobile.gazebo"/>
 </robot>

File: justbaked/src/robdesc/description/robotcore.xacro (robot description, xacro)
@@ -5,5 +5,5 @@
 <!-- Chassis  -->
 <joint name="chassis_joint" type="fixed">
-    <origin xyz="-0.1 0.0 0.1"/>
+    <origin xyz="-0.1 0.0 0.05"/>
     <parent link="base_link"/>
     <child link="chassis"/>
@@ -16,5 +16,5 @@
         </geometry>
         <material name="red">
-            <color rgba="1.0 0.0 0.0 0.9"/>
+            <color rgba="1.0 0.0 0.0 1.0"/>
         </material>
     </visual>

Commit message: lidar upload

File: justbaked/install/robdesc/share/robdesc/description/robot.urdf.xacro (robot description, xacro)
@@ -3,3 +3,4 @@
     <xacro:include filename="robotcore.xacro"/>
     <xacro:include filename="mobile.gazebo"/>
+    <xacro:include filename="rplidar.xacro"/>
 </robot>

File: justbaked/install/robdesc/share/robdesc/description/robotcore.xacro (robot description, xacro)
@@ -123,26 +123,3 @@
     </inertial>
 </link>
-<!-- Lidar -->
-<joint name="lidar_joint" type="continuous">
-    <origin xyz="0.0 0.0 0.3661417" rpy="0.0 0.0 0.0"/>
-    <parent link="chassis"/>
-    <child link="lidar"/>
-    <axis xyz="0.0 0.0 1.0"/>
-</joint>
-<link name="lidar">
-    <visual name="lidar">
-        <origin xyz="0.0 0.0 0.0" rpy="0.0 0.0 0.0"/>
-        <geometry>
-            <cylinder radius="0.229659" length="0.0656168"/>
-        </geometry>
-        <material name="white">
-            <color rgba="1.0 1.0 1.0 1.0"/>
-        </material>
-    </visual>
-    <inertial>
-        <origin xyz="0.0 0.0 0.0" rpy="0.0 0.0 0.0"/>
-        <mass value="1.0"/>
-        <inertia ixx="0.013544611" ixy="0" ixz="0" iyy="0.013544611" iyz="0" izz="0.026371628"/>
-    </inertial>
-</link>
 </robot>
