Commit message: Fixed lidar close range issue and corrected orientation issue

File: justbaked/install/turtlebot4_description/share/turtlebot4_description/urdf/sensors/rplidar.xacro (robot description, xacro)
@@ -6,11 +6,14 @@
     <visual>
       <geometry>
-         <cylinder radius="0.229659" length="0.0656168"/>
+         <cylinder radius="0.07" length="0.02"/>
       </geometry>
+      <material name="White">
+         <color rgba="1.0 1.0 1.0 1.0"/>
+      </material>
     </visual>
     <collision>
-      <origin xyz="0 0 0"/>
+      <origin xyz="0 0 0" rpy="0 0 1.5708"/>
       <geometry>
-         <cylinder radius="0.229659" length="0.0656168"/>
+         <cylinder radius="0.07" length="0.02"/>
       </geometry>
     </collision>
@@ -23,5 +26,5 @@
   <sensor name="lidar_sensor" type="gpu_lidar">
     <topic>scan</topic>
-    <update_rate>1</update_rate>
+    <update_rate>2</update_rate>
     <always_on>true</always_on>
     <visualize>true</visualize>
@@ -42,6 +45,6 @@
       </scan>
       <range>
-        <min>0.2</min>
-        <max>12</max>
+        <min>0</min>
+        <max>3.5</max>
         <resolution>0.013</resolution>
       </range>

File: justbaked/install/turtlebot4_description/share/turtlebot4_description/urdf/standard/robotcore.xacro (robot description, xacro)
@@ -5,5 +5,5 @@
 <!-- Chassis  -->
 <joint name="chassis_joint" type="fixed">
-    <origin xyz="-0.1 0.0 0.05"/>
+    <origin xyz="-0.03048 0.0 0.01524"/>
     <parent link="base_link"/>
     <child link="chassis"/>
@@ -11,7 +11,7 @@
 <link name="chassis">
     <visual name="chassis">
-        <origin xyz="0.0 0.0 0.16666665" rpy="0.0 0.0 0.0"/>
+        <origin xyz="0.0 0.0 0.05" rpy="0.0 0.0 0.0"/>
         <geometry>
-            <box size="1.0 0.8 0.3333333"/>
+            <box size="0.305 0.24384 0.1015999"/>
         </geometry>
         <material name="red">
@@ -22,9 +22,9 @@
         <origin xyz="0.0 0.0 0.05" rpy="0.0 0.0 0.0"/>
         <geometry>
-            <box size="1.0 1.0 0.3333333"/>
+            <box size="0.305 0.305 0.1015999"/>
         </geometry>
     </collision>
     <inertial>
-        <origin xyz="0.0 0.0 0.16666665" rpy="0.0 0.0 0.0"/>
+        <origin xyz="0.0 0.0 0.05" rpy="0.0 0.0 0.0"/>
         <mass value="10.0"/>
         <inertia ixx="0.625924" ixy="0" ixz="0" iyy="1.36667" iyz="0" izz="0.92592"/>
@@ -33,5 +33,5 @@
 <!-- Front left wheel -->
 <joint name="front_left_wheel_joint" type="continuous">
-    <origin xyz="0.4 0.45 0.05" rpy="${pi/2} 0.0 0.0"/>
+    <origin xyz="0.12192 0.13716 0.01524" rpy="${pi/2} 0.0 0.0"/>
     <parent link="chassis"/>
     <child link="front_left_wheel"/>
@@ -42,5 +42,5 @@
         <origin xyz="0.0 0.0 0.0" rpy="0.0 0.0 0.0"/>
         <geometry>
-            <cylinder radius="0.1" length="0.1"/>
+            <cylinder radius="0.03048" length="0.03048"/>
         </geometry>
         <material name="black">
@@ -56,5 +56,5 @@
 <!-- Rear left wheel -->
 <joint name="rear_left_wheel_joint" type="continuous">
-    <origin xyz="-0.4 0.45 0.05" rpy="${pi/2} 0.0 0.0"/>
+    <origin xyz="-0.12192 0.13716 0.01524" rpy="${pi/2} 0.0 0.0"/>
     <parent link="chassis"/>
     <child link="rear_left_wheel"/>
@@ -65,5 +65,5 @@
         <origin xyz="0.0 0.0 0.0" rpy="0.0 0.0 0.0"/>
         <geometry>
-            <cylinder radius="0.1" length="0.1"/>
+            <cylinder radius="0.03048" length="0.03048"/>
         </geometry>
         <material name="black">
@@ -79,5 +79,5 @@
 <!-- Front right wheel -->
 <joint name="front_right_wheel_joint" type="continuous">
-    <origin xyz="0.4 -0.45 0.05" rpy="${pi/2} 0.0 0.0"/>
+    <origin xyz="0.12192 -0.13716 0.01524" rpy="${pi/2} 0.0 0.0"/>
     <parent link="chassis"/>
     <child link="front_right_wheel"/>
@@ -88,5 +88,5 @@
         <origin xyz="0.0 0.0 0.0" rpy="0.0 0.0 0.0"/>
         <geometry>
-            <cylinder radius="0.1" length="0.1"/>
+            <cylinder radius="0.03048" length="0.03048"/>
         </geometry>
         <material name="black">
@@ -102,5 +102,5 @@
 <!-- Rear right wheel -->
 <joint name="rear_right_wheel_joint" type="continuous">
-    <origin xyz="-0.4 -0.45 0.05" rpy="${pi/2} 0.0 0.0"/>
+    <origin xyz="-0.12192 -0.13716 0.01524" rpy="${pi/2} 0.0 0.0"/>
     <parent link="chassis"/>
     <child link="rear_right_wheel"/>
@@ -111,5 +111,5 @@
         <origin xyz="0.0 0.0 0.0" rpy="0.0 0.0 0.0"/>
         <geometry>
-            <cylinder radius="0.1" length="0.1"/>
+            <cylinder radius="0.03048" length="0.03048"/>
         </geometry>
         <material name="black">

File: justbaked/install/turtlebot4_description/share/turtlebot4_description/urdf/standard/turtlebot4.urdf.xacro (robot description, xacro)
@@ -9,5 +9,5 @@
   <!-- Turtlebot4 sensor definitions -->
   <joint name="${name}_joint" type="fixed">
-    <origin xyz=" 0 0 0.3661417" />
+    <origin xyz=" 0 0 0.11159999016" />
     <parent link="${parent_link}"/>
     <child link="${name}_link"/>
