Commit message: Moving robdesc again. Also removed base_footprint

File: justbaked/src/turtlebot4_description/urdf/standard/turtlebot4.urdf.xacro (robot description, xacro)
@@ -13,11 +13,3 @@
     <child link="${name}_link"/>
   </joint>
-  <!-- Base footprint for navigation -->
-  <link name="base_footprint" />
-  <joint name="base_footprint_joint" type="fixed">
-    <!-- Create3's base_link is already on the ground -->
-    <origin xyz="0 0 0" rpy="0 0 0" />
-    <parent link="base_link" />
-    <child link="base_footprint" />
-  </joint>
 </robot>
