Commit message: Saving progress to revert to previous commit.

File: justbaked/install/turtlebot4_description/share/turtlebot4_description/urdf/standard/turtlebot4.urdf.xacro (robot description, xacro)
@@ -1,15 +1 @@
-<?xml version="1.0" ?>
-<robot name="turtlebot4" xmlns:xacro="http://ros.org/wiki/xacro">
-  <!-- Base create3 model -->
-  <xacro:include filename="$(find turtlebot4_description)/urdf/standard/robotcore.xacro"/>
-  <xacro:include filename="$(find turtlebot4_description)/urdf/sensors/rplidar.xacro" />
-  <!-- Mechanical properties -->
-  <xacro:property name="name"                     value="rplidar"/>
-  <xacro:property name="parent_link"              value="chassis"/>
-  <!-- Turtlebot4 sensor definitions -->
-  <joint name="${name}_joint" type="fixed">
-    <origin xyz=" 0 0 0.11159999016" />
-    <parent link="${parent_link}"/>
-    <child link="${name}_link"/>
-  </joint>
-</robot>
+/home/ieee/justbaked/justbaked/src/turtlebot4_description/urdf/standard/turtlebot4.urdf.xacro
