Commit message: First commit from reset.

File: justbaked/install/turtlebot4_description/share/turtlebot4_description/urdf/lite/robot.urdf.xacro (robot description, xacro)
@@ -1,5 +1 @@
-<?xml version="1.0"?>
-<robot xmlns:xacro="http://www.ros.org/wiki/xacro" name="justbaked">
-    <xacro:include filename="robotcore.xacro"/>
-    <xacro:include filename="rplidar.xacro"/>
-</robot>
+/home/ieee/justbaked/justbaked/src/turtlebot4_description/urdf/lite/robot.urdf.xacro

File: justbaked/install/turtlebot4_description/share/turtlebot4_description/urdf/lite/rplidar.xacro (robot description, xacro)
@@ -1,61 +1 @@
-<robot name="sensor_rplidar" xmlns:xacro="http://ros.org/wiki/xacro">
-    <!-- Lidar -->
-<joint name="lidar_joint" type="continuous">
-    <origin xyz="0.0 0.0 0.3661417" rpy="0.0 0.0 0.0"/>
-    <parent link="chassis"/>
-    <child link="lidar_link"/>
-    <axis xyz="0.0 0.0 1.0"/>
-</joint>
-<link name="lidar_link">
-    <visual name="lidar_link">
-        <origin xyz="0.0 0.0 0.0" rpy="0.0 0.0 0.0"/>
-        <geometry>
-            <cylinder radius="0.229659" length="0.0656168"/>
-        </geometry>
-        <material name="white">
-            <color rgba="1.0 1.0 1.0 1.0"/>
-        </material>
-    </visual>
-	<collision>
-		<origin xyz="0.0 0.0 0.0" rpy="0.0 0.0 0.0"/>
-		<geometry>
-			<cylinder radius="0.229659" length="0.0656168"/>
-		</geometry>
-	</collision>
-    <inertial>
-        <origin xyz="0.0 0.0 0.0" rpy="0.0 0.0 0.0"/>
-        <mass value="1.0"/>
-        <inertia ixx="0.013544611" ixy="0" ixz="0" iyy="0.013544611" iyz="0" izz="0.026371628"/>
-    </inertial>
-		    <gazebo reference="lidar">
-      <sensor name="lidar_sensor" type="gpu_lidar">
-        <topic>scan</topic>
-        <update_rate>10</update_rate>
-        <always_on>true</always_on>
-        <visualize>true</visualize>
-        <lidar>
-          <scan>
-            <horizontal>
-              <samples>720</samples>
-              <resolution>1</resolution>
-              <min_angle>-3.14159</min_angle>
-              <max_angle>3.14159</max_angle>
-            </horizontal>
-            <vertical>
-              <samples>1</samples>
-              <resolution>1</resolution>
-              <min_angle>0</min_angle>
-              <max_angle>0</max_angle>
-            </vertical>
-          </scan>
-          <range>
-            <min>0.2</min>
-            <max>12</max>
-            <resolution>0.013</resolution>
-          </range>
-        </lidar>
-        <gz_frame_id>lidar</gz_frame_id>
-      </sensor>
-    </gazebo>
-</link>
-</robot>
+/home/ieee/justbaked/justbaked/src/turtlebot4_description/urdf/lite/rplidar.xacro

File: justbaked/install/turtlebot4_description/share/turtlebot4_description/urdf/sensors/rplidar.xacro (robot description, xacro)
@@ -1,53 +1 @@
-<?xml version="1.0"?>
-<robot xmlns:xacro="http://ros.org/wiki/xacro">
-<xacro:property name="name"                     value="rplidar"/>
-<xacro:property name="parent_link"              value="chassis"/>
-  <link name="${name}_link">
-    <visual>
-      <geometry>
-         <cylinder radius="0.07" length="0.02"/>
-      </geometry>
-      <material name="White">
-         <color rgba="1.0 1.0 1.0 1.0"/>
-      </material>
-    </visual>
-    <collision>
-      <origin xyz="0 0 0" rpy="0 0 1.5708"/>
-      <geometry>
-         <cylinder radius="0.07" length="0.02"/>
-      </geometry>
-    </collision>
-    <inertial>
-        <origin xyz="0.0 0.0 0.0" rpy="0.0 0.0 0.0"/>
-        <mass value="1.0"/>
-        <inertia ixx="0.013544611" ixy="0" ixz="0" iyy="0.013544611" iyz="0" izz="0.026371628"/>
-    </inertial>
-  </link>
-  <sensor name="lidar_sensor" type="gpu_lidar">
-    <topic>scan</topic>
-    <update_rate>2</update_rate>
-    <always_on>true</always_on>
-    <visualize>true</visualize>
-    <lidar>
-      <scan>
-        <horizontal>
-          <samples>720</samples>
-          <resolution>1</resolution>
-          <min_angle>-3.14159</min_angle>
-          <max_angle>3.14159</max_angle>
-        </horizontal>
-        <vertical>
-          <samples>1</samples>
-          <resolution>1</resolution>
-          <min_angle>0</min_angle>
-          <max_angle>0</max_angle>
-        </vertical>
-      </scan>
-      <range>
-        <min>0</min>
-        <max>3.5</max>
-        <resolution>0.013</resolution>
-      </range>
-    </lidar>
-  </sensor>
-</robot>
+/home/ieee/justbaked/justbaked/src/turtlebot4_description/urdf/sensors/rplidar.xacro

File: justbaked/install/turtlebot4_description/share/turtlebot4_description/urdf/standard/robotcore.xacro (robot description, xacro)
@@ -1,125 +1 @@
-<?xml version="1.0"?>
-<robot xmlns:xacro="http://www.ros.org/wiki/xacro">
-<link name="base_link">
-</link>
-<!-- Chassis  -->
-<joint name="chassis_joint" type="fixed">
-    <origin xyz="-0.03048 0.0 0.01524"/>
-    <parent link="base_link"/>
-    <child link="chassis"/>
-</joint>
-<link name="chassis">
-    <visual name="chassis">
-        <origin xyz="0.0 0.0 0.05" rpy="0.0 0.0 0.0"/>
-        <geometry>
-            <box size="0.305 0.24384 0.1015999"/>
-        </geometry>
-        <material name="red">
-            <color rgba="1.0 0.0 0.0 1.0"/>
-        </material>
-    </visual>
-    <collision>
-        <origin xyz="0.0 0.0 0.05" rpy="0.0 0.0 0.0"/>
-        <geometry>
-            <box size="0.305 0.305 0.1015999"/>
-        </geometry>
-    </collision>
-    <inertial>
-        <origin xyz="0.0 0.0 0.05" rpy="0.0 0.0 0.0"/>
-        <mass value="10.0"/>
-        <inertia ixx="0.625924" ixy="0" ixz="0" iyy="1.36667" iyz="0" izz="0.92592"/>
-    </inertial>
-</link>
-<!-- Front left wheel -->
-<joint name="front_left_wheel_joint" type="continuous">
-    <origin xyz="0.12192 0.13716 0.01524" rpy="${pi/2} 0.0 0.0"/>
-    <parent link="chassis"/>
-    <child link="front_left_wheel"/>
-    <axis xyz="0.0 0.0 1.0"/>
-</joint>
-<link name="front_left_wheel">
-    <visual name="front_left_wheel">
-        <origin xyz="0.0 0.0 0.0" rpy="0.0 0.0 0.0"/>
-        <geometry>
-            <cylinder radius="0.03048" length="0.03048"/>
-        </geometry>
-        <material name="black">
-            <color rgba="0.0 0.0 0.0 1.0"/>
-        </material>
-    </visual>
-    <inertial>
-        <origin xyz="0.0 0.0 0.0" rpy="0.0 0.0 0.0"/>
-        <mass value="1.0"/>
-        <inertia ixx="0.003333333" ixy="0" ixz="0" iyy="0.003333333" iyz="0" izz="0.005"/>
-    </inertial>
-</link>
-<!-- Rear left wheel -->
-<joint name="rear_left_wheel_joint" type="continuous">
-    <origin xyz="-0.12192 0.13716 0.01524" rpy="${pi/2} 0.0 0.0"/>
-    <parent link="chassis"/>
-    <child link="rear_left_wheel"/>
-    <axis xyz="0.0 0.0 1.0"/>
-</joint>
-<link name="rear_left_wheel">
-    <visual name="rear_left_wheel">
-        <origin xyz="0.0 0.0 0.0" rpy="0.0 0.0 0.0"/>
-        <geometry>
-            <cylinder radius="0.03048" length="0.03048"/>
-        </geometry>
-        <material name="black">
-            <color rgba="0.0 0.0 0.0 1.0"/>
-        </material>
-    </visual>
-    <inertial>
-        <origin xyz="0.0 0.0 0.0" rpy="0.0 0.0 0.0"/>
-        <mass value="1.0"/>
-        <inertia ixx="0.003333333" ixy="0" ixz="0" iyy="0.003333333" iyz="0" izz="0.005"/>
-    </inertial>
-</link>
-<!-- Front right wheel -->
-<joint name="front_right_wheel_joint" type="continuous">
-    <origin xyz="0.12192 -0.13716 0.01524" rpy="${pi/2} 0.0 0.0"/>
-    <parent link="chassis"/>
-    <child link="front_right_wheel"/>
-    <axis xyz="0.0 0.0 1.0"/>
-</joint>
-<link name="front_right_wheel">
-    <visual name="front_right_wheel">
-        <origin xyz="0.0 0.0 0.0" rpy="0.0 0.0 0.0"/>
-        <geometry>
-            <cylinder radius="0.03048" length="0.03048"/>
-        </geometry>
-        <material name="black">
-            <color rgba="0.0 0.0 0.0 1.0"/>
-        </material>
-    </visual>
-    <inertial>
-        <origin xyz="0.0 0.0 0.0" rpy="0.0 0.0 0.0"/>
-        <mass value="1.0"/>
-        <inertia ixx="0.003333333" ixy="0" ixz="0" iyy="0.003333333" iyz="0" izz="0.005"/>
-    </inertial>
-</link>
-<!-- Rear right wheel -->
-<joint name="rear_right_wheel_joint" type="continuous">
-    <origin xyz="-0.12192 -0.13716 0.01524" rpy="${pi/2} 0.0 0.0"/>
-    <parent link="chassis"/>
-    <child link="rear_right_wheel"/>
-    <axis xyz="0.0 0.0 1.0"/>
-</joint>
-<link name="rear_right_wheel">
-    <visual name="rear_right_wheel">
-        <origin xyz="0.0 0.0 0.0" rpy="0.0 0.0 0.0"/>
-        <geometry>
-            <cylinder radius="0.03048" length="0.03048"/>
-        </geometry>
-        <material name="black">
-            <color rgba="0.0 0.0 0.0 1.0"/>
-        </material>
-    </visual>
-    <inertial>
-        <origin xyz="0.0 0.0 0.0" rpy="0.0 0.0 0.0"/>
-        <mass value="1.0"/>
-        <inertia ixx="0.003333333" ixy="0" ixz="0" iyy="0.003333333" iyz="0" izz="0.005"/>
-    </inertial>
-</link>
-</robot>
+/home/ieee/justbaked/justbaked/src/turtlebot4_description/urdf/standard/robotcore.xacro

File: justbaked/install/turtlebot4_description/share/turtlebot4_description/urdf/standard/turtlebot4.urdf.xacro (robot description, xacro)
@@ -1,23 +1 @@
-<?xml version="1.0" ?>
-<robot name="turtlebot4" xmlns:xacro="http://ros.org/wiki/xacro">
-  <!-- Base create3 model -->
-  <xacro:include filename="$(find turtlebot4_description)/urdf/standard/robotcore.xacro"/>
-  <xacro:include filename="$(find turtlebot4_description)/urdf/sensors/rplidar.xacro" />
-  <!-- Mechanical properties -->
-  <xacro:property name="name"                     value="rplidar"/>
-  <xacro:property name="parent_link"              value="chassis"/>
-  <!-- Turtlebot4 sensor definitions -->
-  <joint name="${name}_joint" type="fixed">
-    <origin xyz=" 0 0 0.11159999016" />
-    <parent link="${parent_link}"/>
-    <child link="${name}_link"/>
-  </joint>
-  <!-- Base footprint for navigation -->
-  <link name="base_footprint" />
-  <joint name="base_footprint_joint" type="fixed">
-    <!-- Create3's base_link is already on the ground -->
-    <origin xyz="0 0 0" rpy="0 0 0" />
-    <parent link="base_link" />
-    <child link="base_footprint" />
-  </joint>
-</robot>
+/home/ieee/justbaked/justbaked/src/turtlebot4_description/urdf/standard/turtlebot4.urdf.xacro
